Commit message: putting parellel gripper urdf and code

File: pterotactyl/objects/test_objects/1.obj.urdf (robot description, URDF)
Before this commit: robot object.urdf, 1 links, 0 joints
Links:
- link baseLink: geometry collision mesh filename=/home/yz8733/Github/Active-3D-Vision-and-Touch/pterotactyl/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 scale=1 1 1; visual mesh filename=/home/yz8733/Github/Active-3D-Vision-and-Touch/pterotactyl/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 scale=1 1 1
